Commit message: change joint names.
shoulder_yaw_joint   --> joint1
shoulder_pitch_joint --> joint2
elbow_pitch_joint    --> joint3
wrist_pitch_joint    --> joint4
wrist_roll_joint     --> joint5

File: pincher_x100_description/urdf/pincher_x100_full.urdf.xacro (robot description, xacro)
@@ -51,16 +51,16 @@
     </xacro:macro>
     <!-- -->
-    <xacro:PincherTransmission joint_name="shoulder_yaw_joint"   actuator_name="joint1" />
-    <xacro:PincherTransmission joint_name="shoulder_pitch_joint" actuator_name="joint2" />
-    <xacro:PincherTransmission joint_name="elbow_pitch_joint"    actuator_name="joint3" />
-    <xacro:PincherTransmission joint_name="wrist_pitch_joint"    actuator_name="joint4" />
-    <xacro:PincherTransmission joint_name="wrist_roll_joint"     actuator_name="joint5" />
+    <xacro:PincherTransmission joint_name="joint1" actuator_name="joint1" />
+    <xacro:PincherTransmission joint_name="joint2" actuator_name="joint2" />
+    <xacro:PincherTransmission joint_name="joint3" actuator_name="joint3" />
+    <xacro:PincherTransmission joint_name="joint4" actuator_name="joint4" />
+    <xacro:PincherTransmission joint_name="joint5" actuator_name="joint5" />
     <!-- -->
     <!--
-    <xacro:PincherTransmission joint_name="shoulder_yaw_joint"   actuator_name="shoulder_yaw_joint" />
-    <xacro:PincherTransmission joint_name="shoulder_pitch_joint" actuator_name="shoulder_pitch_joint" />
-    <xacro:PincherTransmission joint_name="elbow_pitch_joint"    actuator_name="elbow_pitch_joint" />
-    <xacro:PincherTransmission joint_name="wrist_pitch_joint"    actuator_name="wrist_pitch_joint" />
-    <xacro:PincherTransmission joint_name="wrist_roll_joint"     actuator_name="wrist_roll_joint" />
+    <xacro:PincherTransmission joint_name="joint1" actuator_name="joint1" />
+    <xacro:PincherTransmission joint_name="joint2" actuator_name="shoulder_pitch_joint" />
+    <xacro:PincherTransmission joint_name="joint3" actuator_name="joint3" />
+    <xacro:PincherTransmission joint_name="joint4" actuator_name="joint4" />
+    <xacro:PincherTransmission joint_name="joint5" actuator_name="joint5" />
     -->
     <xacro:if value="${use_camera == 'true'}">
@@ -160,5 +160,5 @@
         </visual>
     </link>
-    <joint name="shoulder_yaw_joint" type="revolute">
+    <joint name="joint1" type="revolute">
         <parent link="pincher_x100_base_link"/>
         <child link="shoulder_yaw_link"/>
@@ -188,5 +188,5 @@
         </visual>
     </link>
-    <joint name="shoulder_pitch_joint" type="revolute">
+    <joint name="joint2" type="revolute">
         <parent link="shoulder_yaw_link"/>
         <child link="shoulder_pitch_link"/>
@@ -217,5 +217,5 @@
         </visual>
     </link>
-    <joint name="elbow_pitch_joint" type="revolute">
+    <joint name="joint3" type="revolute">
         <parent link="shoulder_pitch_link"/>
         <child link="elbow_pitch_link"/>
@@ -245,5 +245,5 @@
         </visual>
     </link>
-    <joint name="wrist_pitch_joint" type="revolute">
+    <joint name="joint4" type="revolute">
         <parent link="elbow_pitch_link"/>
         <child link="wrist_pitch_link"/>
@@ -273,5 +273,5 @@
         </visual>
     </link>
-    <joint name="wrist_roll_joint" type="revolute">
+    <joint name="joint5" type="revolute">
         <parent link="wrist_pitch_link"/>
         <child link="wrist_roll_link"/>
